File: Energy_Meter.kicad_pcb (KiCad board)
At the start: 2 copper layers, 73.7 x 86.4 mm, 70 parts, among them IC1 ATM90E36, IC2 Corriente C, J1 Conn_01x02_Male, J5 TENSION, J6 PROGRAMACION, Q1 BC817, Q2 BC817, SW1 RESET, SW2 PR, U1 ESP32-WROOM-32D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

Commit message: Add files via upload
Parts:
- renumbered J1 to FUENTE1
Connections:
- C6 pad 1: Net-(C6-Pad1) -> +3V3
- C7 pad 1: Net-(C6-Pad1) -> +3V3
- C8 pad 1: Net-(C6-Pad1) -> +3V3
- U2 pad 2: Net-(C6-Pad1) -> +3V3

Commit message: Add files via upload
Parts:
- added H1: MountingHole, MountingHole:MountingHole_2.2mm_M2_Pad_Via, F.Cu at (116.3, 52.3)
- added H2: MountingHole, MountingHole:MountingHole_2.2mm_M2_Pad_Via, F.Cu at (181.3, 52.6)
- added H3: MountingHole, MountingHole:MountingHole_2.2mm_M2_Pad_Via, F.Cu at (181.7, 130.2)
- added H4: MountingHole, MountingHole:MountingHole_2.2mm_M2_Pad_Via, F.Cu at (116.2, 130.3)
Routing:
- net (no net): vias 4 -> 0
Changed lines of the file:
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@@
     (thickness 1.6)
     (drawings 4)
-    (tracks 4)
+    (tracks 0)
     (zones 0)
-    (modules 70)
+    (modules 74)
     (nets 91)
   )
@@
     )
   )
+  (module MountingHole:MountingHole_2.2mm_M2_Pad_Via (layer Top)
+    (at 116.3 52.3)
+    (descr "Mounting Hole 2.2mm, M2")
+    (tags "mounting hole 2.2mm m2")
+    (attr virtual)
+    (fp_text reference H1 (at 0 -3.2) (layer F.SilkS)
+      (effects (font (size 1 1) (thickness 0.15)))
+    )
+    (fp_text value MountingHole (at 0 3.2) (layer F.Fab)
+      (effects (font (size 1 1) (thickness 0.15)))
+    )
+    (fp_text user %R (at 0.3 0) (layer F.Fab)
+      (effects (font (size 1 1) (thickness 0.15)))
+    )
+    (fp_circle (center 0 0) (end 2.2 0) (layer Cmts.User) (width 0.15))
+    (fp_circle (center 0 0) (end 2.45 0) (layer F.CrtYd) (width 0.05))
+    (pad 1 thru_hole circle (at 0 0) (size 4.4 4.4) (drill 2.2) (layers *.Cu *.Mask))
+    (pad 1 thru_hole circle (at 1.65 0) (size 0.7 0.7) (drill 0.4) (layers *.Cu *.Mask))
+    (pad 1 thru_hole circle (at 1.166726 1.166726) (size 0.7 0.7) (drill 0.4) (layers *.Cu *.Mask))
+    (pad 1 thru_hole circle (at 0 1.65) (size 0.7 0.7) (drill 0.4) (layers *.Cu *.Mask))
+    (pad 1 thru_hole circle (at -1.166726 1.166726) (size 0.7 0.7) (drill 0.4) (layers *.Cu *.Mask))
+    (pad 1 thru_hole circle (at -1.65 0) (size 0.7 0.7) (drill 0.4) (layers *.Cu *.Mask))
+    (pad 1 thru_hole circle (at -1.166726 -1.166726) (size 0.7 0.7) (drill 0.4) (layers *.Cu *.Mask))
+    (pad 1 thru_hole circle (at 0 -1.65) (size 0.7 0.7) (drill 0.4) (layers *.Cu *.Mask))
+    (pad 1 thru_hole circle (at 1.166726 -1.166726) (size 0.7 0.7) (drill 0.4) (layers *.Cu *.Mask))
+  )
+  (module MountingHole:MountingHole_2.2mm_M2_Pad_Via (layer Top)
+    (at 181.3 52.6)
+    (descr "Mounting Hole 2.2mm, M2")
+    (tags "mounting hole 2.2mm m2")
+    (attr virtual)
+    (fp_text reference H2 (at 0 -3.2) (layer F.SilkS)
+      (effects (font (size 1 1) (thickness 0.15)))
+    )
+    (fp_text value MountingHole (at 0 3.2) (layer F.Fab)
+      (effects (font (size 1 1) (thickness 0.15)))
+    )
+    (fp_text user %R (at 0.3 0) (layer F.Fab)
+      (effects (font (size 1 1) (thickness 0.15)))
+    )
+    (fp_circle (center 0 0) (end 2.2 0) (layer Cmts.User) (width 0.15))
+    (fp_circle (center 0 0) (end 2.45 0) (layer F.CrtYd) (width 0.05))
+    (pad 1 thru_hole circle (at 0 0) (size 4.4 4.4) (drill 2.2) (layers *.Cu *.Mask))
+    (pad 1 thru_hole circle (at 1.65 0) (size 0.7 0.7) (drill 0.4) (layers *.Cu *.Mask))
+    (pad 1 thru_hole circle (at 1.166726 1.166726) (size 0.7 0.7) (drill 0.4) (layers *.Cu *.Mask))
+    (pad 1 thru_hole circle (at 0 1.65) (size 0.7 0.7) (drill 0.4) (layers *.Cu *.Mask))
+    (pad 1 thru_hole circle (at -1.166726 1.166726) (size 0.7 0.7) (drill 0.4) (layers *.Cu *.Mask))
+    (pad 1 thru_hole circle (at -1.65 0) (size 0.7 0.7) (drill 0.4) (layers *.Cu *.Mask))
+    (pad 1 thru_hole circle (at -1.166726 -1.166726) (size 0.7 0.7) (drill 0.4) (layers *.Cu *.Mask))
+    (pad 1 thru_hole circle (at 0 -1.65) (size 0.7 0.7) (drill 0.4) (layers *.Cu *.Mask))
+    (pad 1 thru_hole circle (at 1.166726 -1.166726) (size 0.7 0.7) (drill 0.4) (layers *.Cu *.Mask))
+  )
+  (module MountingHole:MountingHole_2.2mm_M2_Pad_Via (layer Top)
+    (at 181.65 130.15)
+    (descr "Mounting Hole 2.2mm, M2")
+    (tags "mounting hole 2.2mm m2")
+    (attr virtual)
+    (fp_text reference H3 (at 0 -3.2) (layer F.SilkS)
+      (effects (font (size 1 1) (thickness 0.15)))
+    )
+    (fp_text value MountingHole (at 0 3.2) (layer F.Fab)
+      (effects (font (size 1 1) (thickness 0.15)))
+    )
+    (fp_circle (center 0 0) (end 2.45 0) (layer F.CrtYd) (width 0.05))
+    (fp_circle (center 0 0) (end 2.2 0) (layer Cmts.User) (width 0.15))
+    (fp_text user %R (at 0.3 0) (layer F.Fab)
+      (effects (font (size 1 1) (thickness 0.15)))
+    )
+    (pad 1 thru_hole circle (at 1.166726 -1.166726) (size 0.7 0.7) (drill 0.4) (layers *.Cu *.Mask))
+    (pad 1 thru_hole circle (at 0 -1.65) (size 0.7 0.7) (drill 0.4) (layers *.Cu *.Mask))
+    (pad 1 thru_hole circle (at -1.166726 -1.166726) (size 0.7 0.7) (drill 0.4) (layers *.Cu *.Mask))
+    (pad 1 thru_hole circle (at -1.65 0) (size 0.7 0.7) (drill 0.4) (layers *.Cu *.Mask))
+    (pad 1 thru_hole circle (at -1.166726 1.166726) (size 0.7 0.7) (drill 0.4) (layers *.Cu *.Mask))
+    (pad 1 thru_hole circle (at 0 1.65) (size 0.7 0.7) (drill 0.4) (layers *.Cu *.Mask))
+    (pad 1 thru_hole circle (at 1.166726 1.166726) (size 0.7 0.7) (drill 0.4) (layers *.Cu *.Mask))
+    (pad 1 thru_hole circle (at 1.65 0) (size 0.7 0.7) (drill 0.4) (layers *.Cu *.Mask))
+    (pad 1 thru_hole circle (at 0 0) (size 4.4 4.4) (drill 2.2) (layers *.Cu *.Mask))
+  )
+  (module MountingHole:MountingHole_2.2mm_M2_Pad_Via (layer Top)
+    (at 116.2 130.35)
+    (descr "Mounting Hole 2.2mm, M2")
+    (tags "mounting hole 2.2mm m2")
+    (attr virtual)
+    (fp_text reference H4 (at 0 -3.2) (layer F.SilkS)
+      (effects (font (size 1 1) (thickness 0.15)))
+    )
+    (fp_text value MountingHole (at 0 3.2) (layer F.Fab)
+      (effects (font (size 1 1) (thickness 0.15)))
+    )
+    (fp_circle (center 0 0) (end 2.45 0) (layer F.CrtYd) (width 0.05))
+    (fp_circle (center 0 0) (end 2.2 0) (layer Cmts.User) (width 0.15))
+    (fp_text user %R (at 0.3 0) (layer F.Fab)
+      (effects (font (size 1 1) (thickness 0.15)))
+    )
+    (pad 1 thru_hole circle (at 1.166726 -1.166726) (size 0.7 0.7) (drill 0.4) (layers *.Cu *.Mask))
+    (pad 1 thru_hole circle (at 0 -1.65) (size 0.7 0.7) (drill 0.4) (layers *.Cu *.Mask))
+    (pad 1 thru_hole circle (at -1.166726 -1.166726) (size 0.7 0.7) (drill 0.4) (layers *.Cu *.Mask))
+    (pad 1 thru_hole circle (at -1.65 0) (size 0.7 0.7) (drill 0.4) (layers *.Cu *.Mask))
+    (pad 1 thru_hole circle (at -1.166726 1.166726) (size 0.7 0.7) (drill 0.4) (layers *.Cu *.Mask))
+    (pad 1 thru_hole circle (at 0 1.65) (size 0.7 0.7) (drill 0.4) (layers *.Cu *.Mask))
+    (pad 1 thru_hole circle (at 1.166726 1.166726) (size 0.7 0.7) (drill 0.4) (layers *.Cu *.Mask))
+    (pad 1 thru_hole circle (at 1.65 0) (size 0.7 0.7) (drill 0.4) (layers *.Cu *.Mask))
+    (pad 1 thru_hole circle (at 0 0) (size 4.4 4.4) (drill 2.2) (layers *.Cu *.Mask))
+  )
   (gr_line (start 112.014 134.366) (end 112.014 48.006) (layer Edge.Cuts) (width 0.05))
   (gr_line (start 185.674 134.366) (end 112.014 134.366) (layer Edge.Cuts) (width 0.05))
   (gr_line (start 185.674 48.006) (end 185.674 134.366) (layer Edge.Cuts) (width 0.05))
   (gr_line (start 112.014 48.006) (end 185.674 48.006) (layer Edge.Cuts) (width 0.05))
-  (via (at 119.634 55.118) (size 3.3) (drill 2.8) (layers Top Bottom) (net 0))
-  (via (at 175.514 55.626) (size 3.3) (drill 2.8) (layers Top Bottom) (net 0))
-  (via (at 175.514 126.746) (size 3.3) (drill 2.8) (layers Top Bottom) (net 0))
-  (via (at 119.634 126.746) (size 3.3) (drill 2.8) (layers Top Bottom) (net 0))
 )

Commit message: Add files via upload
Parts:
- removed FUENTE1: Conn_01x02_Male, Connector_Molex:Molex_KK-254_AE-6410-02A_1x02_P2.54mm_Vertical
- added FUENTE: Conn_01x02_Male, Connector_Molex:Molex_KK-254_AE-6410-02A_1x02_P2.54mm_Vertical, F.Cu at (84.2, 71.8)
- moved C21 38.2 mm to (144.7, 120.2)
- moved Y1 36.3 mm to (140.6, 118.3), turned to 90 degrees
- moved C22 35.0 mm to (144.7, 112.5), turned to 90 degrees
- moved C18 35.0 mm to (118.6, 115.8)
- moved R27 34.9 mm to (138.3, 93.4)
- moved R14 34.9 mm to (118.0, 122.8)
- moved C19 34.9 mm to (125.7, 115.7)
- moved R23 34.9 mm to (115.2, 115.8)
- moved R24 34.9 mm to (122.2, 115.8)
- moved H2 34.8 mm to (146.9, 58.5)
- moved C10 34.8 mm to (102.5, 94.8)
- moved C11 34.8 mm to (102.5, 104.8)
- moved C13 34.8 mm to (121.4, 122.8)
- moved C2 34.8 mm to (115.0, 105.4)
- moved C7 34.8 mm to (86.8, 79.8)
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Routing:
- net GND: track 0.00 -> 470.4 mm, vias 0 -> 6
- net +3V3: track 0.00 -> 197.7 mm
- net /ENABLE: track 0.00 -> 70.8 mm, vias 0 -> 3
- net /IDO: track 0.00 -> 65.4 mm, vias 0 -> 1
- net ICN: track 0.00 -> 43.4 mm, vias 0 -> 2
- net ICP: track 0.00 -> 40.5 mm, vias 0 -> 3
- net Net-(IC1-Pad37): track 0.00 -> 38.9 mm, vias 0 -> 2
- net Net-(J6-Pad2): track 0.00 -> 36.1 mm
- net IBP: track 0.00 -> 32.8 mm, vias 0 -> 2
- net Net-(IC1-Pad38): track 0.00 -> 32.2 mm, vias 0 -> 2
- net VAP: track 0.00 -> 31.0 mm, vias 0 -> 2
- net IBN: track 0.00 -> 31.0 mm, vias 0 -> 2
- net /CONFIGURACION/IB-: track 0.00 -> 30.5 mm, vias 0 -> 3
- net IAN: track 0.00 -> 30.4 mm, vias 0 -> 2
- net /CONFIGURACION/IB+: track 0.00 -> 29.7 mm, vias 0 -> 2
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- added copper zone on F.Cu, net GND
Other:
- board text added: "Especificaciones: Layers: 2 Delivery Format: Single PCB PCB Thickness: 1.6 PCB Color: RED Surface Finish: HASL Copper Weight: 1 OZ Material Type: FR4-Standard Tg 130-140C Castellated Holes: NO"
- board text added: "Fabricante: https://jlcpcb.com/#"

Commit message: Add files via upload
Parts:
- added G***: LOGO, ATM90E36_Breakout:fiuba, F.Cu at (140.2, 130.4)
- renumbered IC2 to IC1
Routing:
- added copper zone on B.Cu, net GND
Changed lines of the file:
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@@
     (tracks 594)
     (zones 0)
-    (modules 74)
+    (modules 75)
     (nets 91)
   )
@@
     (34 B.Paste user)
     (35 F.Paste user)
-    (36 B.SilkS user hide)
+    (36 B.SilkS user)
     (37 F.SilkS user)
     (38 B.Mask user hide)
-    (39 F.Mask user hide)
+    (39 F.Mask user)
     (40 Dwgs.User user hide)
-    (41 Cmts.User user hide)
+    (41 Cmts.User user)
     (42 Eco1.User user hide)
     (43 Eco2.User user hide)
@@
       (outputformat 1)
       (mirror false)
-      (drillshape 1)
+      (drillshape 0)
       (scaleselection 1)
-      (outputdirectory ""))
+      (outputdirectory "Gerbers/"))
   )
   (net 0 "")
@@
     (add_net VCP)
   )
+  (module ATM90E36_Breakout:fiuba (layer Top)
+    (at 140.2 130.4)
+    (fp_text reference G*** (at -0.2 5) (layer Cmts.User)
+      (effects (font (size 1.524 1.524) (thickness 0.3)))
+    )
+    (fp_text value LOGO (at 0.75 0) (layer Dwgs.User)
+      (effects (font (size 1.524 1.524) (thickness 0.3)))
+    )
+    (fp_poly (pts (xy 2.117835 -2.693253) (xy 2.332461 -2.494197) (xy 2.219116 -2.288739) (xy 1.820005 -2.321724)
+      (xy 1.464438 -2.379524) (xy 1.474772 -2.26298) (xy 1.875364 -1.90012) (xy 1.997397 -1.797565)
+      (xy 2.492602 -1.330398) (xy 2.607674 -1.006104) (xy 2.432554 -0.700037) (xy 1.968215 -0.383442)
+      (xy 1.406259 -0.27526) (xy 0.951477 -0.382606) (xy 0.802105 -0.64339) (xy 0.998629 -0.906117)
+      (xy 1.336842 -0.879575) (xy 1.773954 -0.881042) (xy 1.842125 -1.102868) (xy 1.545609 -1.382439)
+      (xy 1.321255 -1.475474) (xy 0.889575 -1.810255) (xy 0.835243 -2.27759) (xy 1.118672 -2.675205)
+      (xy 1.58193 -2.807369) (xy 2.117835 -2.693253)) (layer F.SilkS) (width 0.01))
+    (fp_poly (pts (xy -0.278903 -2.7297) (xy 0.15827 -2.272632) (xy 0.441164 -1.749338) (xy 0.395409 -1.337881)
+      (xy 0.15827 -0.93579) (xy -0.455606 -0.383) (xy -1.075638 -0.267369) (xy -1.546837 -0.297078)
+      (xy -1.78181 -0.478149) (xy -1.86267 -0.948498) (xy -1.871579 -1.604211) (xy -1.336842 -1.604211)
+      (xy -1.270532 -1.017152) (xy -1.023672 -0.838247) (xy -0.868948 -0.853005) (xy -0.482917 -1.171161)
+      (xy -0.401053 -1.604211) (xy -0.573613 -2.182874) (xy -0.868948 -2.355417) (xy -1.202541 -2.30043)
+      (xy -1.328478 -1.880807) (xy -1.336842 -1.604211) (xy -1.871579 -1.604211) (xy -1.853891 -2.395626)
+      (xy -1.746083 -2.79028) (xy -1.466042 -2.92609) (xy -1.075638 -2.941053) (xy -0.278903 -2.7297)) (layer F.SilkS) (width 0.01))
+    (fp_poly (pts (xy -3.308363 -2.703857) (xy -3.215239 -2.111312) (xy -3.208421 -1.871579) (xy -3.163579 -1.171891)
+      (xy -2.982333 -0.862656) (xy -2.673684 -0.802106) (xy -2.23922 -0.690139) (xy -2.138948 -0.534737)
+      (xy -2.371282 -0.347009) (xy -2.931074 -0.267389) (xy -2.941053 -0.267369) (xy -3.41588 -0.296576)
+      (xy -3.652658 -0.476155) (xy -3.734152 -0.944045) (xy -3.743158 -1.604211) (xy -3.695065 -2.366803)
+      (xy -3.5721 -2.850837) (xy -3.47579 -2.941053) (xy -3.308363 -2.703857)) (layer F.SilkS) (width 0.01))
+    (fp_poly (pts (xy 2.298365 1.183816) (xy 2.517457 1.508192) (xy 2.587695 2.176063) (xy 2.346239 2.719254)
+      (xy 1.884745 2.941052) (xy 1.421456 2.71765) (xy 1.269303 2.444291) (xy 1.266815 2.005263)
+      (xy 1.60421 2.005263) (xy 1.695734 2.507731) (xy 1.871579 2.673684) (xy 2.072566 2.444875)
+      (xy 2.138947 2.005263) (xy 2.047424 1.502795) (xy 1.871579 1.336842) (xy 1.670591 1.56565)
+      (xy 1.60421 2.005263) (xy 1.266815 2.005263) (xy 1.265767 1.8204) (xy 1.519364 1.339909)
+      (xy 1.905197 1.096491) (xy 2.298365 1.183816)) (layer F.SilkS) (width 0.01))
+    (fp_poly (pts (xy 0.713342 1.275789) (xy 0.792809 1.727047) (xy 0.636818 2.171715) (xy 0.506192 2.290273)
+      (xy 0.384159 2.531643) (xy 0.573034 2.703011) (xy 0.721029 2.87829) (xy 0.374159 2.936503)
+      (xy 0.33421 2.936958) (xy -0.135314 2.845399) (xy -0.267369 2.689463) (xy -0.073019 2.327356)
+      (xy 0 2.272631) (xy 0.243326 1.88693) (xy 0.267368 1.706336) (xy 0.12267 1.449073)
+      (xy -0.041311 1.496057) (xy -0.22427 1.52757) (xy -0.159216 1.378152) (xy 0.253915 1.093346)
+      (xy 0.416832 1.069473) (xy 0.713342 1.275789)) (layer F.SilkS) (width 0.01))
+    (fp_poly (pts (xy -0.910056 1.183816) (xy -0.690964 1.508192) (xy -0.620726 2.176063) (xy -0.862182 2.719254)
+      (xy -1.323676 2.941052) (xy -1.786965 2.71765) (xy -1.939118 2.444291) (xy -1.941606 2.005263)
+      (xy -1.604211 2.005263) (xy -1.512687 2.507731) (xy -1.336842 2.673684) (xy -1.135855 2.444875)
+      (xy -1.069474 2.005263) (xy -1.160997 1.502795) (xy -1.336842 1.336842) (xy -1.53783 1.56565)
+      (xy -1.604211 2.005263) (xy -1.941606 2.005263) (xy -1.942654 1.8204) (xy -1.689057 1.339909)
+      (xy -1.303224 1.096491) (xy -0.910056 1.183816)) (layer F.SilkS) (width 0.01))
+    (fp_poly (pts (xy -2.495079 1.275789) (xy -2.415613 1.727047) (xy -2.571603 2.171715) (xy -2.702229 2.290273)
+      (xy -2.824262 2.531643) (xy -2.635387 2.703011) (xy -2.487392 2.87829) (xy -2.834262 2.936503)
+      (xy -2.874211 2.936958) (xy -3.343735 2.845399) (xy -3.47579 2.689463) (xy -3.28144 2.327356)
+      (xy -3.208421 2.272631) (xy -2.965095 1.88693) (xy -2.941053 1.706336) (xy -3.085751 1.449073)
+      (xy -3.249732 1.496057) (xy -3.432691 1.52757) (xy -3.367637 1.378152) (xy -2.954506 1.093346)
+      (xy -2.791589 1.069473) (xy -2.495079 1.275789)) (layer F.SilkS) (width 0.01))
+  )
   (module Crystal:Crystal_HC49-4H_Vertical (layer Top)
     (at 140.55 118.35 90)
@@
     (tags "CMS SOT")
     (attr smd)
-    (fp_text reference U2 (at 0 -4.5 90) (layer F.SilkS)
+    (fp_text reference U2 (at 3.196 -4.412 90) (layer F.SilkS)
       (effects (font (size 1 1) (thickness 0.15)))
     )
@@
     (tags capacitor)
     (attr smd)
-    (fp_text reference C11 (at 0 -1.65) (layer F.SilkS)
+    (fp_text reference C11 (at -0.0935 -1.65) (layer F.SilkS)
       (effects (font (size 1 1) (thickness 0.15)))
     )
@@
     (tags capacitor)
     (attr smd)
-    (fp_text reference C14 (at 0 -1.65) (layer F.SilkS)
+    (fp_text reference C14 (at 0.044 1.536) (layer F.SilkS)
       (effects (font (size 1 1) (thickness 0.15)))
     )
@@
     (tags "3.5mm audio cui horizontal jack stereo")
     (attr smd)
-    (fp_text reference IC2 (at 0 -9.9 90) (layer F.SilkS)
+    (fp_text reference IC1 (at 0 -9.9 90) (layer F.SilkS)
       (effects (font (size 1 1) (thickness 0.15)))
     )
@@
     (descr "Molex KK-254 Interconnect System, old/engineering part number: AE-6410-04A example for new part number: 22-27-2041, 4 Pins (http://www.molex.com/pdm_docs/sd/022272021_sd.pdf), generated with kicad-footprint-generator")
     (tags "connector Molex KK-254 side entry")
-    (fp_text reference J5 (at 3.81 -4.12) (layer F.SilkS)
+    (fp_text reference J5 (at -2.952 0.072) (layer F.SilkS)
       (effects (font (size 1 1) (thickness 0.15)))
     )
@@
     (descr "Through hole straight pin header, 1x05, 2.54mm pitch, single row")
     (tags "Through hole pin header THT 1x05 2.54mm single row")
-    (fp_text reference J6 (at 0 -2.33) (layer F.SilkS)
+    (fp_text reference J6 (at 0 -2.95) (layer F.SilkS)
       (effects (font (size 1 1) (thickness 0.15)))
     )
@@
     (descr "tactile push button, 6x6mm e.g. PHAP33xx series, height=4.3mm")
     (tags "tact sw push 6mm")
-    (fp_text reference SW1 (at 3.25 -2) (layer F.SilkS)
+    (fp_text reference SW1 (at 3.156 -2.336) (layer F.SilkS)
       (effects (font (size 1 1) (thickness 0.15)))
     )
@@
     (descr "tactile push button, 6x6mm e.g. PHAP33xx series, height=4.3mm")
     (tags "tact sw push 6mm")
-    (fp_text reference SW2 (at 3.25 -2) (layer F.SilkS)
+    (fp_text reference SW2 (at 3.25 -2.236) (layer F.SilkS)
       (effects (font (size 1 1) (thickness 0.15)))
     )
@@
     (pad 1 thru_hole circle (at 0 0) (size 4.4 4.4) (drill 2.2) (layers *.Cu *.Mask))
   )
-  (gr_text "Fabricante: \n\nhttps://jlcpcb.com/#" (at 170.95 57.45) (layer F.SilkS)
+  (gr_text "Fabricante: \n\nhttps://jlcpcb.com/#" (at 170.95 57.45) (layer Cmts.User)
     (effects (font (size 3 3) (thickness 0.15)) (justify left))
   )
-  (gr_text "Especificaciones: \nLayers: 2\nDelivery Format: Single PCB\nPCB Thickness: 1.6\nPCB Color: RED\nSurface Finish: HASL\nCopper Weight: 1 OZ\nMaterial Type: FR4-Standard Tg 130-140C\nCastellated Holes: NO\n" (at 169.3 87.6) (layer F.SilkS)
+  (gr_text "Especificaciones: \nLayers: 2\nDelivery Format: Single PCB\nPCB Thickness: 1.6\nPCB Color: RED\nSurface Finish: HASL\nCopper Weight: 1 OZ\nMaterial Type: FR4-Standard Tg 130-140C\nCastellated Holes: NO\n" (at 169.3 87.6) (layer Cmts.User)
     (effects (font (size 2 2) (thickness 0.25)) (justify left))
   )
@@
       )
     )
+  )
+  (zone (net 1) (net_name GND) (layer Bottom) (hatch edge 0.508)
+    (connect_pads (clearance 0.508))
+    (min_thickness 0.254)
+    (fill yes (arc_segments 32) (thermal_gap 0.508) (thermal_bridge_width 0.508))
+    (polygon
+      (pts
+        (xy 150.6 139.4) (xy 77.7 139.4) (xy 77.7 53.9) (xy 150.6 53.9)
+      )
+    )

Commit message: Add files via upload
Parts:
- removed Power1: LED, LED_SMD:LED_0805_2012Metric
- added POWER: LED, LED_SMD:LED_0805_2012Metric, F.Cu at (98.1, 61.4)
- renumbered D1 to WIFI
Routing:
- net Net-(IC1-Pad41): track 10.6 -> 17.1 mm
Other:
- board text added: "5v"
- board text added: "GND"

Commit message: Add files via upload
Parts:
- added F1: Fiducial, Fiducial:Fiducial_0.5mm_Mask1.5mm, F.Cu at (90.3, 135.2)
- added F2: Fiducial, Fiducial:Fiducial_0.5mm_Mask1.5mm, F.Cu at (139.8, 61.6)
- added F3: Fiducial, Fiducial:Fiducial_0.5mm_Mask1.5mm, F.Cu at (139.8, 107.3)
- CON1: renamed from FUENTE; value Conn_01x02_Male -> Fuente
- LED2: renamed from POWER; value LED -> Power
- SW2: value PR -> PROG
- moved R28 7.61 mm to (94.4, 62.8), turned to 0 degrees
- moved LED1 2.56 mm to (91.2, 59.0)
- moved LED2 2.47 mm to (97.4, 59.0)
- moved H2 2.03 mm to (147.4, 56.5)
- moved H1 1.76 mm to (81.4, 56.5)
- moved H4 0.53 mm to (81.4, 136.5)
- moved H3 0.51 mm to (147.4, 136.5)
- moved SW1 0.21 mm to (139.8, 67.8)
- renumbered WIFI to LED1, IC1 to U2, U2 to U3
Connections:
- net /CONFIGURACION/VA renamed Net-(J5-Pad4)
- net /CONFIGURACION/VB renamed Net-(J5-Pad3)
- net /CONFIGURACION/VC renamed Net-(J5-Pad2)
- net IAN renamed /IAN
- net IAP renamed /IAP
- net IBN renamed /IBN
- net IBP renamed /IBP
- net ICN renamed /ICN
- net ICP renamed /ICP
- net VAP renamed /VAP
- net VBP renamed /VBP
- net VCP renamed /VCP
Routing:
- net +3V3: track 197.6 -> 208.7 mm
- net Net-(LED1-Pad2): track 11.6 -> 4.36 mm
- net Net-(R28-Pad2): track 27.2 -> 31.3 mm, vias 2 -> 0
- net GND: track 470.4 -> 468.1 mm
- net /ENABLE: track 70.8 -> 72.0 mm, vias 3 -> 2
- net Net-(LED2-Pad2): track 12.8 -> 13.8 mm
- removed copper zone on B.Cu, net GND
- removed copper zone on F.Cu, net GND
Other:
- board size 73.7 x 86.4 mm -> 74.9 x 87.6 mm
- board text added: "Especificaciones: Layers: 2 Delivery Format: Single PCB PCB Thickness: 1.6 PCB Color: RED Surface Finish: HASL Copper Weight: 1 OZ Material Type: FR4-Standard Tg 130-140C Castellated Holes: NO Ancho de pistas: 0.25, 0.3 y 0.5 mm Grillas: 10 y 50 mils Vía: 0.40 y 0.80 mils"
- board text removed: "Especificaciones: Layers: 2 Delivery Format: Single PCB PCB Thickness: 1.6 PCB Color: RED Surface Finish: HASL Copper Weight: 1 OZ Material Type: FR4-Standard Tg 130-140C Castellated Holes: NO"

Commit message: Add files via upload
Connections:
- net Net-(R1-Pad2) renamed /MISO
- net Net-(R2-Pad2) renamed /MOSI
- net Net-(R3-Pad2) renamed /CLK
- net Net-(R4-Pad2) renamed /CS
Routing:
- added copper zone on B.Cu, net GND
- added copper zone on F.Cu, net GND
Other:
- rule trace_min: 0.1524 -> 0.25
- board text added: "IND. ARG"

Commit message: Add files via upload
Routing:
- net Net-(R30-Pad2): track 17.1 -> 9.09 mm
- net /MISO: track 29.0 -> 26.0 mm
- net /MOSI: track 21.0 -> 19.9 mm
- net +3V3: track 208.7 -> 209.7 mm
- net /CLK: track 32.2 -> 33.2 mm
- net /CS: track 38.9 -> 39.6 mm
Other:
- net class Default: clearance 0.1524 -> 0.25
- rule trace_clearance: 0.1524 -> 0.25
