File: Energy_Meter.kicad_pcb (KiCad board)
At the start: 2 copper layers, 74.9 x 87.6 mm, 78 parts, among them CON1 Fuente, IC1 Corriente C, J5 TENSION, J6 PROGRAMACION, Q1 BC817, Q2 BC817, SW1 RESET, SW2 PROG, U1 ESP32-WROOM-32D, U2 ATM90E36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

Commit message: Add files via upload
Parts:
- renumbered LED1 to D1, LED2 to D2
Routing:
- net +3V3: track 209.7 -> 210.7 mm
Other:
- board text added: "Especificaciones: Layers: 2 Delivery Format: Single PCB PCB Thickness: 1.6 PCB Color: RED Surface Finish: HASL Copper Weight: 1 OZ Material Type: FR4-Standard Tg 130-140C Castellated Holes: NO Ancho de pistas: 0.25, 0.3 y 0.5 mm Grillas: 0.2540 y 1.2700 mm Vía: 0.8 y 3.3 mm"
- board text removed: "Especificaciones: Layers: 2 Delivery Format: Single PCB PCB Thickness: 1.6 PCB Color: RED Surface Finish: HASL Copper Weight: 1 OZ Material Type: FR4-Standard Tg 130-140C Castellated Holes: NO Ancho de pistas: 0.25, 0.3 y 0.5 mm Grillas: 10 y 50 mils Vía: 0.40 y 0.80 mils"

Commit message: Add files via upload
Parts:
- renumbered IA1 to J1, IB1 to J2, IC1 to J3, CON1 to J4
