File: Energy_Meter.sch (KiCad schematic (older format))
At the start: 30 parts, among them IC1 ATM90E36, J1 Conn_01x02_Male, J6 PROGRAMACION, Q1 BC817, Q2 BC817, U1 ESP32-WROOM-32D, U2 LD1117S18TR_SOT223, Y1 Crystal

Commit message: Add files via upload
Parts:
- added D1: Conexión, LED_SMD:LED_0805_2012Metric, symbol Device:LED
- added Power1: LED, LED_SMD:LED_0805_2012Metric, symbol Device:LED
- added R28, R29: 560, Resistor_SMD:R_0805_2012Metric, symbol Device:R
- added R30, R31: 10K, Resistor_SMD:R_0805_2012Metric, symbol Device:R
- added R32: 50R, Resistor_SMD:R_0805_2012Metric, symbol Device:R
- added SW1: RESET, Button_Switch_THT:SW_PUSH_6mm_H4.3mm, symbol Switch:SW_Push
- added SW2: PR, Button_Switch_THT:SW_PUSH_6mm_H4.3mm, symbol Switch:SW_Push
- C1, C3, C4, C7: value C -> 100nF
- C18, C19, C20: value C -> 18nF
- C2, C5, C6: value CP -> 10uF
- C21, C22: value C -> 22pF
- C8: value C -> 47nF
- R1, R2, R26, R27, R3, R4: value R -> 10K
- R23, R24, R25: value R -> 1K
- Y1: value Crystal -> 16.384MHz
Connections:
- net +3V3: now also R30.1, R31.1
- net ENABLE: now also R31.2, SW1.1
- net GND: now also D1.1 (K), Power1.1 (K), R32.1, SW1.2
- net IDO: now also SW2.1
- net at IC1.41 (~RESET): now also R30.2
- net at U1.12 (IO27): now also R28.2
- net at U1.6 (IO34): now also R29.2
- new net: D1.2 (A), R28.1
- new net: Power1.2 (A), R29.1
- new net: R32.2, SW2.2
- no-connect marks 41 -> 38

Commit message: Add files via upload
Parts:
- renumbered J1 to FUENTE1
Connections:
- net +3V3: now also C6.1, C7.1, C8.1, U2.2 (VO)
Changed lines of the file:
@@
 	4200 3650 4250 3650
-Wire Wire Line
-	4300 3650 4300 3800
 Wire Wire Line
 	4250 2650 4250 3650
@@
 Wire Wire Line
 	5450 2250 5700 2250
-$Comp
-L Connector:Conn_01x02_Male J1
-U 1 1 5EE1A71F
-P 1200 1350
-F 0 "J1" H 1308 1531 50  0000 C CNN
-F 1 "Conn_01x02_Male" H 1308 1440 50  0000 C CNN
-F 2 "Connector_Molex:Molex_KK-254_AE-6410-02A_1x02_P2.54mm_Vertical" H 1200 1350 50  0001 C CNN
-F 3 "~" H 1200 1350 50  0001 C CNN
-	1    1200 1350
-	1    0    0    -1
-$EndComp
 Wire Wire Line
 	2250 4400 3200 4400
@@
 	1400 1950 2000 1950
 Connection ~ 2000 1950
-Wire Wire Line
-	1400 1350 2000 1350
 $Comp
 L power:+5V #PWR0107
@@
 Wire Wire Line
 	8500 1700 9200 1700
+Wire Wire Line
+	1400 1350 1750 1350
+$Comp
+L Connector:Conn_01x02_Male FUENTE1
+U 1 1 5EE1A71F
+P 1200 1350
+F 0 "FUENTE1" H 1308 1531 50  0000 C CNN
+F 1 "Conn_01x02_Male" H 1308 1440 50  0000 C CNN
+F 2 "Connector_Molex:Molex_KK-254_AE-6410-02A_1x02_P2.54mm_Vertical" H 1200 1350 50  0001 C CNN
+F 3 "~" H 1200 1350 50  0001 C CNN
+	1    1200 1350
+	1    0    0    -1
+$EndComp
+$Comp
+L power:PWR_FLAG #FLG0101
+U 1 1 5EDB805A
+P 1750 1050
+F 0 "#FLG0101" H 1750 1125 50  0001 C CNN
+F 1 "PWR_FLAG" H 1750 1223 50  0000 C CNN
+F 2 "" H 1750 1050 50  0001 C CNN
+F 3 "~" H 1750 1050 50  0001 C CNN
+	1    1750 1050
+	1    0    0    -1
+$EndComp
+$Comp
+L power:PWR_FLAG #FLG0102
+U 1 1 5EDD028A
+P 2000 2100
+F 0 "#FLG0102" H 2000 2175 50  0001 C CNN
+F 1 "PWR_FLAG" H 2000 2273 50  0000 C CNN
+F 2 "" H 2000 2100 50  0001 C CNN
+F 3 "~" H 2000 2100 50  0001 C CNN
+	1    2000 2100
+	-1   0    0    1
+$EndComp
+Wire Wire Line
+	1750 1050 1750 1350
+Connection ~ 1750 1350
+Wire Wire Line
+	1750 1350 2000 1350
+Wire Wire Line
+	2000 2100 2000 1950
+Wire Wire Line
+	4300 3650 4300 3800
+$Comp
+L power:+3.3V #PWR0112
+U 1 1 5EDF845A
+P 4050 1050
+F 0 "#PWR0112" H 4050 900 50  0001 C CNN
+F 1 "+3.3V" H 4065 1223 50  0000 C CNN
+F 2 "" H 4050 1050 50  0001 C CNN
+F 3 "" H 4050 1050 50  0001 C CNN
+	1    4050 1050
+	1    0    0    -1
+$EndComp
+Wire Wire Line
+	4050 1050 4050 1350
 $EndSCHEMATC

Commit message: Add files via upload
Parts:
- added H1, H2, H3, H4: MountingHole, MountingHole:MountingHole_2.2mm_M2_Pad_Via, symbol Mechanical:MountingHole
Changed lines of the file:
@@
 Wire Wire Line
 	4050 1050 4050 1350
+$Comp
+L Mechanical:MountingHole H1
+U 1 1 5EDB88BD
+P 1100 2700
+F 0 "H1" H 1200 2746 50  0000 L CNN
+F 1 "MountingHole" H 1200 2655 50  0000 L CNN
+F 2 "MountingHole:MountingHole_2.2mm_M2_Pad_Via" H 1100 2700 50  0001 C CNN
+F 3 "~" H 1100 2700 50  0001 C CNN
+	1    1100 2700
+	1    0    0    -1
+$EndComp
+$Comp
+L Mechanical:MountingHole H3
+U 1 1 5EDB90A9
+P 1900 2700
+F 0 "H3" H 2000 2746 50  0000 L CNN
+F 1 "MountingHole" H 2000 2655 50  0000 L CNN
+F 2 "MountingHole:MountingHole_2.2mm_M2_Pad_Via" H 1900 2700 50  0001 C CNN
+F 3 "~" H 1900 2700 50  0001 C CNN
+	1    1900 2700
+	1    0    0    -1
+$EndComp
+$Comp
+L Mechanical:MountingHole H2
+U 1 1 5EDB940D
+P 1100 2950
+F 0 "H2" H 1200 2996 50  0000 L CNN
+F 1 "MountingHole" H 1200 2905 50  0000 L CNN
+F 2 "MountingHole:MountingHole_2.2mm_M2_Pad_Via" H 1100 2950 50  0001 C CNN
+F 3 "~" H 1100 2950 50  0001 C CNN
+	1    1100 2950
+	1    0    0    -1
+$EndComp
+$Comp
+L Mechanical:MountingHole H4
+U 1 1 5EDB973F
+P 1900 2950
+F 0 "H4" H 2000 2996 50  0000 L CNN
+F 1 "MountingHole" H 2000 2905 50  0000 L CNN
+F 2 "MountingHole:MountingHole_2.2mm_M2_Pad_Via" H 1900 2950 50  0001 C CNN
+F 3 "~" H 1900 2950 50  0001 C CNN
+	1    1900 2950
+	1    0    0    -1
+$EndComp
 $EndSCHEMATC

Commit message: Add files via upload
Other:
- note added: "ATM90E36\n"
- note added: "CLK\n"
- note added: "CS"
- note added: "FUENTE 5V\n"
- note added: "MISO"
- note added: "MOSI"
- note added: "SALIDA: 3.3V"
- note added: "SPI"
- moved on the sheet: C18, C19, C2, C5, C6, C7, R1, R2, R23, R24, R25, R4

Commit message: Add files via upload
Parts:
- added F1, F2, F3: Fiducial, Fiducial:Fiducial_0.5mm_Mask1.5mm, symbol Mechanical:Fiducial
- CON1: renamed from FUENTE1; value Conn_01x02_Male -> Fuente
- LED2: renamed from Power1; value LED -> Power
- Q1: Mouser (none) -> 771-BC817K-40HVL; descripción (none) -> Bipolar Transistors - BJT NPN Epitaxial Silicon Transistor
- Q2: Descripción (none) -> Bipolar Transistors - BJT NPN Epitaxial Silicon Transistor; Mouser (none) -> 771-BC817K-16HR
- SW2: value PR -> PROG
- U1: Descripción (none) -> Módulo ESP32 wifi + bluetooth; Mouser (none) -> 356-ESP32WRM32E132PH
- U2: renamed from IC1; Descripción (none) -> Circuito integrado medidor de energía; Mouser (none) -> 556-ATM90E36A-AU-Y
- U3: renamed from U2; Descripción (none) -> Regulador de 3.3v; Mouser (none) -> 511-LD1117AS18
- Y1: Descripción (none) -> Crystals 16384kHz 20pF With Thermistor; Digikey (none) -> XC2790TR-ND
- renumbered D1 to LED1
Connections:
- net CS: now reaches R4.2, U1.19 (SCS/CMD), U2.37 (~CS)
- net CLK: now reaches R3.2, U1.20 (SCK/CLK), U2.38 (SCLK)
- net MISO: now reaches R1.2, U1.21 (SDO/SD0), U2.39 (SDO)
- net MOSI: now reaches R2.2, U1.22 (SDI/SD1), U2.40 (SDI)
Other:
- note added: "CIRCUITO INTEGRTADO\n ENERGY METER"
- note added: "ESP32-WROOM\nWIFI - BLUETOOTH"
- note added: "Fiduciales"
- note added: "Orificios de Montaje\n"
- note removed: "CLK\n"
- note removed: "CS"
- note removed: "MISO"
- note removed: "MOSI"
- note removed: "SPI"
- moved on the sheet: C1, C18, C19, C2, C20, C21, C22, C3, C4, C5, C6, C7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

Commit message: Add files via upload
Changed lines of the file:
@@
 Title "Módem Energy Meter"
 Date "5/5/2020"
-Rev "8/6/2020"
+Rev "5/7/2020"
 Comp "Autor: Del Sancio Leonardo Daniel"
 Comment1 "Alumno Rev: Yapura Albert"
@@
 U 1 1 5ED95B59
 P 7850 3000
-F 0 "U1" H 7850 4581 50  0000 C CNN
+F 0 "U1" H 8100 4400 50  0000 C CNN
 F 1 "ESP32-WROOM-32D" H 7750 3700 50  0000 C CNN
 F 2 "RF_Module:ESP32-WROOM-32" H 7850 1500 50  0001 C CNN
@@
 Wire Wire Line
 	4150 3900 4150 3750
-Wire Wire Line
-	4150 3750 4200 3750
-Wire Wire Line
-	4200 2750 4200 3750
-Connection ~ 4200 3750
-Wire Wire Line
-	4200 3750 4250 3750
 Wire Wire Line
 	4750 3500 4750 3900
@@
 	2200 3950 2200 3550
 Wire Wire Line
-	2200 3550 2850 3550
+	2200 3550 2500 3550
 Wire Wire Line
 	3750 3400 3900 3400
@@
 Wire Wire Line
 	3900 3000 3900 2750
-Connection ~ 3900 2750
-Wire Wire Line
-	3900 2750 4200 2750
 NoConn ~ 5250 4400
 NoConn ~ 5250 4900
@@
 Wire Wire Line
 	2200 4500 3150 4500
-Wire Wire Line
-	3650 2750 3650 3550
-Wire Wire Line
-	3650 3550 3650 3900
-Connection ~ 3650 3550
-Connection ~ 2850 3550
-Wire Wire Line
-	2850 3550 3650 3550
 $Comp
 L power:+3.3V #PWR0101
@@
 L power:+3.3V #PWR0108
 U 1 1 5EDC4044
-P 3900 2550
-F 0 "#PWR0108" H 3900 2400 50  0001 C CNN
-F 1 "+3.3V" H 3915 2723 50  0000 C CNN
-F 2 "" H 3900 2550 50  0001 C CNN
-F 3 "" H 3900 2550 50  0001 C CNN
-	1    3900 2550
-	1    0    0    -1
-$EndComp
-Wire Wire Line
-	3900 2550 3900 2750
+P 3650 2650
+F 0 "#PWR0108" H 3650 2500 50  0001 C CNN
+F 1 "+3.3V" H 3665 2823 50  0000 C CNN
+F 2 "" H 3650 2650 50  0001 C CNN
+F 3 "" H 3650 2650 50  0001 C CNN
+	1    3650 2650
+	1    0    0    -1
+$EndComp
 $Comp
 L power:+3.3V #PWR0109
 U 1 1 5EDC66D6
-P 7850 1050
-F 0 "#PWR0109" H 7850 900 50  0001 C CNN
-F 1 "+3.3V" H 7865 1223 50  0000 C CNN
-F 2 "" H 7850 1050 50  0001 C CNN
-F 3 "" H 7850 1050 50  0001 C CNN
-	1    7850 1050
+P 7850 1200
+F 0 "#PWR0109" H 7850 1050 50  0001 C CNN
+F 1 "+3.3V" H 7865 1373 50  0000 C CNN
+F 2 "" H 7850 1200 50  0001 C CNN
+F 3 "" H 7850 1200 50  0001 C CNN
+	1    7850 1200
 	1    0    0    -1
 $EndComp
@@
 $EndComp
 Wire Wire Line
-	7850 1050 7850 1250
-Wire Wire Line
 	6600 1350 6600 1250
-Wire Wire Line
-	6600 1250 7850 1250
-Connection ~ 7850 1250
-Wire Wire Line
-	7850 1250 7850 1600
 Wire Wire Line
 	6600 1800 7250 1800
@@
 Text Label 8550 2100 0    50   ~ 0
 RX
-Text Label 8550 1800 0    50   ~ 0
+Text Label 8650 1800 0    50   ~ 0
 IDO
 Wire Wire Line
@@
 Wire Wire Line
 	8350 1800 8450 1800
-Connection ~ 8450 1800
-Wire Wire Line
-	8450 1800 8800 1800
 $Sheet
 S 9850 800  1100 1900
@@
 	4650 2350 5000 2350
 Connection ~ 5000 2350
+$Comp
+L power:+3.3V #PWR0118
+U 1 1 5F62ECEA
+P 2500 3400
+F 0 "#PWR0118" H 2500 3250 50  0001 C CNN
+F 1 "+3.3V" H 2515 3573 50  0000 C CNN
+F 2 "" H 2500 3400 50  0001 C CNN
+F 3 "" H 2500 3400 50  0001 C CNN
+	1    2500 3400
+	1    0    0    -1
+$EndComp
+Wire Wire Line
+	3650 2750 3650 3900
+Wire Wire Line
+	2500 3400 2500 3550
+Connection ~ 2500 3550
+Wire Wire Line
+	2500 3550 2850 3550
+$Comp
+L power:+3.3V #PWR0119
+U 1 1 5F63A3E7
+P 6600 1250
+F 0 "#PWR0119" H 6600 1100 50  0001 C CNN
+F 1 "+3.3V" H 6615 1423 50  0000 C CNN
+F 2 "" H 6600 1250 50  0001 C CNN
+F 3 "" H 6600 1250 50  0001 C CNN
+	1    6600 1250
+	1    0    0    -1
+$EndComp
+Wire Wire Line
+	4150 3750 4200 3750
+$Comp
+L power:+3.3V #PWR0120
+U 1 1 5F63A7EA
+P 4200 3650
+F 0 "#PWR0120" H 4200 3500 50  0001 C CNN
+F 1 "+3.3V" H 4215 3823 50  0000 C CNN
+F 2 "" H 4200 3650 50  0001 C CNN
+F 3 "" H 4200 3650 50  0001 C CNN
+	1    4200 3650
+	1    0    0    -1
+$EndComp
+Wire Wire Line
+	3650 2650 3650 2750
+Connection ~ 3650 2750
+Wire Wire Line
+	4200 3650 4200 3750
+Connection ~ 4200 3750
+Wire Wire Line
+	4200 3750 4250 3750
+Wire Wire Line
+	7850 1200 7850 1600
+Wire Wire Line
+	8450 1800 8800 1800
+Connection ~ 8450 1800
 $EndSCHEMATC

Commit message: Add files via upload
Parts:
- renumbered LED1 to D1, LED2 to D2
Other:
- note removed: "ATM90E36\n"
- note removed: "CIRCUITO INTEGRTADO\n ENERGY METER"
- note removed: "ESP32-WROOM\nWIFI - BLUETOOTH"
- moved on the sheet: C1
Changed lines of the file:
@@
 Title "Módem Energy Meter"
 Date "5/5/2020"
-Rev "5/7/2020"
+Rev "15/7/2020"
 Comp "Autor: Del Sancio Leonardo Daniel"
-Comment1 "Alumno Rev: Yapura Albert"
+Comment1 "Alumno Rev: Yapura Alberto"
 Comment2 "Prof. Rev: Diego Brengi"
-Comment3 ""
+Comment3 "License: CC BY 4.0"
 Comment4 ""
 $EndDescr
@@
 P 7850 3000
 F 0 "U1" H 8100 4400 50  0000 C CNN
-F 1 "ESP32-WROOM-32D" H 7750 3700 50  0000 C CNN
+F 1 "ESP32-WROOM-32D" V 7900 3250 50  0000 C CNN
 F 2 "RF_Module:ESP32-WROOM-32" H 7850 1500 50  0001 C CNN
 F 3 "https://www.espressif.com/sites/default/files/documentation/esp32-wroom-32d_esp32-wroom-32u_datasheet_en.pdf" H 7550 3050 50  0001 C CNN
@@
 Wire Wire Line
 	3150 4400 2850 4400
-Wire Wire Line
-	2850 4400 2850 3550
 $Comp
 L Device:C C3
@@
 L Device:C C1
 U 1 1 5EDC35DE
-P 2200 4100
-F 0 "C1" H 2315 4146 50  0000 L CNN
-F 1 "100nF" H 2315 4055 50  0000 L CNN
-F 2 "Capacitor_SMD:C_0805_2012Metric" H 2238 3950 50  0001 C CNN
-F 3 "~" H 2200 4100 50  0001 C CNN
-	1    2200 4100
-	1    0    0    -1
-$EndComp
-Wire Wire Line
-	2200 4250 2200 4500
-Wire Wire Line
-	2200 3950 2200 3550
-Wire Wire Line
-	2200 3550 2500 3550
+P 2350 4100
+F 0 "C1" H 2465 4146 50  0000 L CNN
+F 1 "100nF" H 2465 4055 50  0000 L CNN
+F 2 "Capacitor_SMD:C_0805_2012Metric" H 2388 3950 50  0001 C CNN
+F 3 "~" H 2350 4100 50  0001 C CNN
+	1    2350 4100
+	1    0    0    -1
+$EndComp
 Wire Wire Line
 	3750 3400 3900 3400
@@
 P 4250 4900
 F 0 "U2" H 5294 4903 59  0000 L CNN
-F 1 "ATM90E36" H 5294 4798 59  0000 L CNN
+F 1 "ATM90E36" H 4000 4850 59  0000 L CNN
 F 2 "Package_QFP:TQFP-48_7x7mm_P0.5mm" H 4250 4900 50  0001 C CNN
 F 3 "https://ww1.microchip.com/downloads/en/DeviceDoc/Atmel-46004-SE-M90E36A-Datasheet.pdf" H 4250 4900 50  0001 C CNN
@@
 NoConn ~ 7250 2000
 NoConn ~ 7250 2100
-Wire Wire Line
-	2200 4500 3150 4500
 $Comp
 L power:+3.3V #PWR0101
@@
 L power:GND #PWR0105
 U 1 1 5ED9EB47
-P 2350 6100
-F 0 "#PWR0105" H 2350 5850 50  0001 C CNN
-F 1 "GND" H 2355 5927 50  0000 C CNN
-F 2 "" H 2350 6100 50  0001 C CNN
-F 3 "" H 2350 6100 50  0001 C CNN
-	1    2350 6100
+P 2350 4600
+F 0 "#PWR0105" H 2350 4350 50  0001 C CNN
+F 1 "GND" H 2355 4427 50  0000 C CNN
+F 2 "" H 2350 4600 50  0001 C CNN
+F 3 "" H 2350 4600 50  0001 C CNN
+	1    2350 4600
 	1    0    0    -1
 $EndComp
@@
 	9000 4000 9250 4000
 $Comp
-L Device:LED LED1
+L Device:LED D1
 U 1 1 5EEBF10E
 P 9400 3700
-F 0 "LED1" H 9400 3500 50  0000 C CNN
+F 0 "D1" H 9400 3500 50  0000 C CNN
 F 1 "Conexión" H 9400 3600 50  0000 C CNN
 F 2 "LED_SMD:LED_0805_2012Metric" H 9400 3700 50  0001 C CNN
@@
 $EndComp
 $Comp
-L Device:LED LED2
+L Device:LED D2
 U 1 1 5EEBF72F
 P 9400 4000
-F 0 "LED2" H 9400 4100 50  0000 C CNN
+F 0 "D2" H 9400 4100 50  0000 C CNN
 F 1 "Power" H 9400 4200 50  0000 C CNN
 F 2 "LED_SMD:LED_0805_2012Metric" H 9400 4000 50  0001 C CNN
@@
 	1    0    0    -1
 $EndComp
-Text Notes 4000 5050 0    50   ~ 0
-ATM90E36\n
 Wire Wire Line
 	3300 6550 3950 6550
@@
 Wire Wire Line
 	2350 5850 2350 6000
-Connection ~ 2350 6000
 Wire Wire Line
 	2350 6000 2750 6000
-Wire Wire Line
-	2350 6100 2350 6000
 Wire Wire Line
 	4750 3500 5950 3500
@@
 Wire Wire Line
 	9750 2550 9850 2550
-Wire Wire Line
-	2050 6000 2050 4500
-Wire Wire Line
-	2050 4500 2200 4500
-Connection ~ 2200 4500
-Wire Wire Line
-	2050 6000 2350 6000
-Text Notes 3800 5250 0    50   ~ 0
-CIRCUITO INTEGRTADO\n    ENERGY METER
-Text Notes 7400 4000 0    50   ~ 0
-ESP32-WROOM\nWIFI - BLUETOOTH
 Text Label 7150 3000 2    50   ~ 0
 MISO
@@
 L power:+3.3V #PWR0118
 U 1 1 5F62ECEA
-P 2500 3400
-F 0 "#PWR0118" H 2500 3250 50  0001 C CNN
-F 1 "+3.3V" H 2515 3573 50  0000 C CNN
-F 2 "" H 2500 3400 50  0001 C CNN
-F 3 "" H 2500 3400 50  0001 C CNN
-	1    2500 3400
+P 2850 3950
+F 0 "#PWR0118" H 2850 3800 50  0001 C CNN
+F 1 "+3.3V" H 2865 4123 50  0000 C CNN
+F 2 "" H 2850 3950 50  0001 C CNN
+F 3 "" H 2850 3950 50  0001 C CNN
+	1    2850 3950
 	1    0    0    -1
 $EndComp
 Wire Wire Line
 	3650 2750 3650 3900
-Wire Wire Line
-	2500 3400 2500 3550
-Connection ~ 2500 3550
-Wire Wire Line
-	2500 3550 2850 3550
 $Comp
 L power:+3.3V #PWR0119
@@
 	8450 1800 8800 1800
 Connection ~ 8450 1800
+$Comp
+L power:+3.3V #PWR0121
+U 1 1 5F107EE9
+P 2350 3950
+F 0 "#PWR0121" H 2350 3800 50  0001 C CNN
+F 1 "+3.3V" H 2365 4123 50  0000 C CNN
+F 2 "" H 2350 3950 50  0001 C CNN
+F 3 "" H 2350 3950 50  0001 C CNN
+	1    2350 3950
+	1    0    0    -1
+$EndComp
+Wire Wire Line
+	2350 4500 3150 4500
+Wire Wire Line
+	2350 4250 2350 4500
+Wire Wire Line
+	2350 4500 2350 4600
+Connection ~ 2350 4500
+Wire Wire Line
+	2850 3950 2850 4400
+$Comp
+L power:GND #PWR0122
+U 1 1 5F13324C
+P 2750 6050
+F 0 "#PWR0122" H 2750 5800 50  0001 C CNN
+F 1 "GND" H 2755 5877 50  0000 C CNN
+F 2 "" H 2750 6050 50  0001 C CNN
+F 3 "" H 2750 6050 50  0001 C CNN
+	1    2750 6050
+	1    0    0    -1
+$EndComp
+Wire Wire Line
+	2750 6000 2750 6050
 $EndSCHEMATC

Commit message: Add files via upload
Parts:
- renumbered CON1 to J4
Changed lines of the file:
@@
 	1150 1350 1500 1350
 $Comp
-L Connector:Conn_01x02_Male CON1
+L Connector:Conn_01x02_Male J4
 U 1 1 5EE1A71F
 P 950 1350
-F 0 "CON1" H 1058 1531 50  0000 C CNN
+F 0 "J4" H 1058 1531 50  0000 C CNN
 F 1 "Fuente" H 1058 1440 50  0000 C CNN
 F 2 "Connector_Molex:Molex_KK-254_AE-6410-02A_1x02_P2.54mm_Vertical" H 950 1350 50  0001 C CNN
@@
 Wire Wire Line
 	1750 1800 1750 1950
-Text Notes 3300 1250 0    50   ~ 0
+Text Notes 3400 1050 0    50   ~ 0
 SALIDA: 3.3V
 Text Notes 750  1050 0    50   ~ 0
