File: conectores.sch (KiCad schematic (older format))
At the start: 31 parts, among them J2 CORRIENTE A, J3 CORRIENTE B, J4 CORRIENTE C, J5 TENSION

Commit message: Add files via upload
Parts:
- removed J2: CORRIENTE A, Connector_Audio:Jack_3.5mm_PJ31060-I_Horizontal, symbol Connector:AudioJack3_Ground
- removed J3: CORRIENTE B, Capacitor_SMD:CP_Elec_5x5.3, symbol Connector:AudioJack3_Ground
- removed J4: CORRIENTE C, Capacitor_SMD:CP_Elec_5x5.3, symbol Connector:AudioJack3_Ground
- added IA1: Corriente A, Connector_Audio:Jack_3.5mm_CUI_SJ-3523-SMT_Horizontal, symbol Connector:AudioJack3
- added IB1: Corriente B, Connector_Audio:Jack_3.5mm_CUI_SJ-3523-SMT_Horizontal, symbol Connector:AudioJack3
- added IC2: Corriente C, Connector_Audio:Jack_3.5mm_CUI_SJ-3523-SMT_Horizontal, symbol Connector:AudioJack3
- C10, C11, C12, C13, C14, C15, C16, C17, C9: value C -> 18nF
- R10, R12, R14, R17, R18, R21, R22, R8, R9: value R -> 1K
- R11, R13, R7: value R -> 100K
- R15, R16, R19, R20, R5, R6: value R -> 2.4
Connections:
- wire segments 101 -> 98

Commit message: Add files via upload
Other:
- note added: "CONECTOR JACK SJ-352X-SMT"
- note added: "Configuración de Corriente"
- note removed: "Configuración de Corriente\n"
Changed lines of the file:
@@
 Wire Bus Line
 	750  3100 10650 3100
-Text Notes 4900 900  0    50   ~ 0
+Text Notes 4250 900  0    150  Italic 30
 Configuración de Tensión
-Text Notes 5000 3450 0    50   ~ 0
-Configuración de Corriente\n
 $Comp
 L Connector:AudioJack3 IA1
@@
 	1    0    0    -1
 $EndComp
+Text Notes 2850 7200 0    80   ~ 0
+CONECTOR JACK  SJ-352X-SMT
+Text Notes 4150 3500 0    150  Italic 30
+Configuración de Corriente
 $EndSCHEMATC

Commit message: Add files via upload
Parts:
- renumbered IC2 to IC1
Connections:
- net VA: no longer names the net of J5.4 (Pin_4), R7.1
- net VB: no longer names the net of J5.3 (Pin_3), R11.1
- net VC: no longer names the net of J5.2 (Pin_2), R13.1
Other:
- moved on the sheet: C10, C11, C12, C13, C14, C15, C16, C17, C9, IA1, IB1, IC1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

Commit message: Add files via upload
Parts:
- renumbered IA1 to J1, IB1 to J2, IC1 to J3
Changed lines of the file:
@@
 Configuración de Tensión
 $Comp
-L Connector:AudioJack3 IA1
+L Connector:AudioJack3 J1
 U 1 1 5EDFB80D
 P 2250 7000
-F 0 "IA1" H 2232 7325 50  0000 C CNN
+F 0 "J1" H 2232 7325 50  0000 C CNN
 F 1 "Corriente A" H 2232 7234 50  0000 C CNN
 F 2 "Connector_Audio:Jack_3.5mm_CUI_SJ-3523-SMT_Horizontal" H 2250 7000 50  0001 C CNN
@@
 $EndComp
 $Comp
-L Connector:AudioJack3 IB1
+L Connector:AudioJack3 J2
 U 1 1 5EDFC470
 P 3550 7000
-F 0 "IB1" H 3532 7325 50  0000 C CNN
+F 0 "J2" H 3532 7325 50  0000 C CNN
 F 1 "Corriente B" H 3532 7234 50  0000 C CNN
 F 2 "Connector_Audio:Jack_3.5mm_CUI_SJ-3523-SMT_Horizontal" H 3550 7000 50  0001 C CNN
@@
 $EndComp
 $Comp
-L Connector:AudioJack3 IC1
+L Connector:AudioJack3 J3
 U 1 1 5EDFCA1A
 P 4750 7000
-F 0 "IC1" H 4732 7325 50  0000 C CNN
+F 0 "J3" H 4732 7325 50  0000 C CNN
 F 1 "Corriente C" H 4732 7234 50  0000 C CNN
 F 2 "Connector_Audio:Jack_3.5mm_CUI_SJ-3523-SMT_Horizontal" H 4750 7000 50  0001 C CNN
